File: PCB_Final_Project.kicad_pcb (KiCad board)
At the start: 2 copper layers, 49 x 43.3 mm, 22 parts, among them P1 Power_Con, Q1 BC148, Q2 BC158, Q3 AC187, Q4 AC188

Commit message: Final Project
Other:
- net class power added: clearance 0.5, trace_width 0.3, via_dia 0.6, via_drill 0.4
Changed lines of the file:
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@@
     (add_net "Net-(Q4-Pad3)")
+  )
+  (net_class power ""
+    (clearance 0.5)
+    (trace_width 0.3)
+    (via_dia 0.6)
+    (via_drill 0.4)
+    (uvia_dia 0.3)
+    (uvia_drill 0.1)
   )
   (module Potentiometers:Potentiometer_Alps_RK097_Single_Vertical (layer F.Cu)
@@
     (descr TO-11-3)
     (tags TO-11-3)
-    (fp_text reference Q4 (at 6.39318 -4.25704 180) (layer F.SilkS)
-      (effects (font (size 1 1) (thickness 0.15)))
-    )
+    (fp_text reference Q4 (at 7.57936 -3.37058 180) (layer F.SilkS)
+      (effects (font (size 1 1) (thickness 0.15)))
+    )
